File: hardware/schematic.brd (EAGLE design)
At the start: 124 x 80 mm, 72 parts, among them IC1 TL494CN, IC2 7805TV, IC3 7815TV, IC4 LM4558N, IC5 TINY13-20PU, Q1 IPP086N10N3G, Q3 BS170, U1 IR2101

Commit message: Initial commit
Parts:
- C11, C12: value 2m2 -> 2m2 50V
- C13, C14, C15, C18: value 100n -> 100n 50V
- C17, C9: value 10n -> 10n 50V
- R22: value 8k2 -> 8k2 0,5W
Changed lines of the file:
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@@
 <attribute name="VALUE" x="30.606" y="67.738" size="1.27" layer="27" ratio="10" rot="R180"/>
 </element>
-<element name="C11" library="rcl" library_urn="urn:adsk.eagle:library:334" package="E7,5-18" package3d_urn="urn:adsk.eagle:package:23379/1" value="2m2" x="61.16" y="52.31" smashed="yes" rot="R270">
+<element name="C11" library="rcl" library_urn="urn:adsk.eagle:library:334" package="E7,5-18" package3d_urn="urn:adsk.eagle:package:23379/1" value="2m2 50V" x="61.16" y="52.31" smashed="yes" rot="R270">
 <attribute name="NAME" x="66.24" y="44.309" size="1.778" layer="25" ratio="10" rot="R270"/>
 <attribute name="POPULARITY" value="6" x="51" y="-15" size="1.778" layer="27" rot="R270" display="off"/>
@@
 <attribute name="VALUE" x="56.8674" y="57.39" size="1.778" layer="27" ratio="10" rot="R270"/>
 </element>
-<element name="C12" library="rcl" library_urn="urn:adsk.eagle:library:334" package="E7,5-18" package3d_urn="urn:adsk.eagle:package:23379/1" value="2m2" x="80.16" y="52.45" smashed="yes" rot="R270">
+<element name="C12" library="rcl" library_urn="urn:adsk.eagle:library:334" package="E7,5-18" package3d_urn="urn:adsk.eagle:package:23379/1" value="2m2 50V" x="80.16" y="52.45" smashed="yes" rot="R270">
 <attribute name="NAME" x="85.24" y="44.449" size="1.778" layer="25" ratio="10" rot="R270"/>
 <attribute name="POPULARITY" value="6" x="70" y="8" size="1.778" layer="27" rot="R270" display="off"/>
@@
 <attribute name="VALUE" x="75.8674" y="57.53" size="1.778" layer="27" ratio="10" rot="R270"/>
 </element>
-<element name="C13" library="capacitor-wima" library_urn="urn:adsk.eagle:library:116" package="C2.5-2" package3d_urn="urn:adsk.eagle:package:5415/1" value="100n" x="70.09" y="60.2" smashed="yes">
+<element name="C13" library="capacitor-wima" library_urn="urn:adsk.eagle:library:116" package="C2.5-2" package3d_urn="urn:adsk.eagle:package:5415/1" value="100n 50V" x="70.09" y="60.2" smashed="yes">
 <attribute name="NAME" x="68.439" y="61.724" size="1.27" layer="25" ratio="10"/>
 <attribute name="POPULARITY" value="28" x="112" y="-16" size="1.778" layer="27" display="off"/>
 <attribute name="VALUE" x="68.439" y="57.406" size="1.27" layer="27" ratio="10"/>
 </element>
-<element name="C14" library="capacitor-wima" library_urn="urn:adsk.eagle:library:116" package="C2.5-2" package3d_urn="urn:adsk.eagle:package:5415/1" value="100n" x="94.8" y="17.74" smashed="yes" rot="R90">
+<element name="C14" library="capacitor-wima" library_urn="urn:adsk.eagle:library:116" package="C2.5-2" package3d_urn="urn:adsk.eagle:package:5415/1" value="100n 50V" x="94.8" y="17.74" smashed="yes" rot="R90">
 <attribute name="NAME" x="93.276" y="16.089" size="1.27" layer="25" ratio="10" rot="R90"/>
 <attribute name="POPULARITY" value="28" x="171" y="66" size="1.778" layer="27" rot="R90" display="off"/>
 <attribute name="VALUE" x="97.594" y="16.089" size="1.27" layer="27" ratio="10" rot="R90"/>
 </element>
-<element name="C15" library="capacitor-wima" library_urn="urn:adsk.eagle:library:116" package="C2.5-2" package3d_urn="urn:adsk.eagle:package:5415/1" value="100n" x="78" y="7.61" smashed="yes" rot="R270">
+<element name="C15" library="capacitor-wima" library_urn="urn:adsk.eagle:library:116" package="C2.5-2" package3d_urn="urn:adsk.eagle:package:5415/1" value="100n 50V" x="78" y="7.61" smashed="yes" rot="R270">
 <attribute name="NAME" x="79.524" y="9.261" size="1.27" layer="25" ratio="10" rot="R270"/>
 <attribute name="POPULARITY" value="28" x="1.8" y="-47" size="1.778" layer="27" rot="R270" display="off"/>
@@
 <attribute name="VALUE" x="110.406" y="32.611" size="1.27" layer="27" ratio="10" rot="R270"/>
 </element>
-<element name="C17" library="capacitor-wima" library_urn="urn:adsk.eagle:library:116" package="C2.5-2" package3d_urn="urn:adsk.eagle:package:5415/1" value="10n" x="110.24" y="59.18" smashed="yes" rot="R180">
+<element name="C17" library="capacitor-wima" library_urn="urn:adsk.eagle:library:116" package="C2.5-2" package3d_urn="urn:adsk.eagle:package:5415/1" value="10n 50V" x="110.24" y="59.18" smashed="yes" rot="R180">
 <attribute name="NAME" x="111.891" y="57.656" size="1.27" layer="25" ratio="10" rot="R180"/>
 <attribute name="POPULARITY" value="28" x="95" y="143" size="1.778" layer="27" rot="R180" display="off"/>
 <attribute name="VALUE" x="111.891" y="61.974" size="1.27" layer="27" ratio="10" rot="R180"/>
 </element>
-<element name="C18" library="capacitor-wima" library_urn="urn:adsk.eagle:library:116" package="C2.5-2" package3d_urn="urn:adsk.eagle:package:5415/1" value="100n" x="103.69" y="19.2" smashed="yes">
+<element name="C18" library="capacitor-wima" library_urn="urn:adsk.eagle:library:116" package="C2.5-2" package3d_urn="urn:adsk.eagle:package:5415/1" value="100n 50V" x="103.69" y="19.2" smashed="yes">
 <attribute name="NAME" x="102.039" y="20.724" size="1.27" layer="25" ratio="10"/>
 <attribute name="POPULARITY" value="28" x="171" y="-57" size="1.778" layer="27" display="off"/>
@@
 <attribute name="VALUE" x="22.466" y="47.738" size="1.27" layer="27" ratio="10" rot="R180"/>
 </element>
-<element name="C9" library="capacitor-wima" library_urn="urn:adsk.eagle:library:116" package="C2.5-2" package3d_urn="urn:adsk.eagle:package:5415/1" value="10n" x="100.8" y="57.56" smashed="yes" rot="R90">
+<element name="C9" library="capacitor-wima" library_urn="urn:adsk.eagle:library:116" package="C2.5-2" package3d_urn="urn:adsk.eagle:package:5415/1" value="10n 50V" x="100.8" y="57.56" smashed="yes" rot="R90">
 <attribute name="NAME" x="99.276" y="55.909" size="1.27" layer="25" ratio="10" rot="R90"/>
 <attribute name="POPULARITY" value="28" x="177" y="149" size="1.778" layer="27" rot="R90" display="off"/>
@@
 <attribute name="VALUE" x="52.1144" y="13.5774" size="0.9906" layer="27" ratio="10"/>
 </element>
-<element name="R22" library="rcl" library_urn="urn:adsk.eagle:library:334" package="0204/7" package3d_urn="urn:adsk.eagle:package:23498/2" value="8k2" x="97.58" y="12.06" smashed="yes">
+<element name="R22" library="rcl" library_urn="urn:adsk.eagle:library:334" package="0204/7" package3d_urn="urn:adsk.eagle:package:23498/2" value="8k2 0,5W" x="97.58" y="12.06" smashed="yes">
 <attribute name="NAME" x="95.04" y="13.3554" size="0.9906" layer="25" ratio="10"/>
 <attribute name="POPULARITY" value="79" x="156" y="-87" size="1.778" layer="27" display="off"/>
